Commit message: 112

File: install/dojo/share/dojo/description/gazebo_control.xacro (robot description, xacro)
@@ -6,6 +6,6 @@
             <left_joint>left_wheel_joint</left_joint>
             <right_joint>right_wheel_joint</right_joint>
-            <wheel_separation>0.28</wheel_separation>
-            <wheel_diameter>0.065</wheel_diameter>
+            <wheel_separation>0.25</wheel_separation>
+            <wheel_diameter>0.085</wheel_diameter>
             <!-- limits -->
             <max_wheel_torque>200</max_wheel_torque>

File: install/dojo/share/dojo/description/lidar.xacro (robot description, xacro)
@@ -4,5 +4,5 @@
         <parent link="chassis"/>
         <child link="laser_frame"/>
-        <origin xyz="0.0 0.0 0.08" rpy="0.0 0.0 0.0"/>
+        <origin xyz="0.1 0.0 0.08" rpy="0.0 0.0 0.0"/>
     </joint>
     <link name="laser_frame">

File: install/dojo/share/dojo/description/robot.urdf.xacro (robot description, xacro)
@@ -1,13 +1,7 @@
 <?xml version="1.0"?>
 <robot xmlns:xacro="http://www.ros.org/wiki/xacro"  name="robot">
-    <xacro:arg name = "use_ros2_control" default="true"/>
-    <xacro:arg name="sim_mode" default="true"/>
     <xacro:include filename="robot_core.xacro"/>
-    <xacro:if value = "$(arg use_ros2_control)">
-        <xacro:include filename="ros2_control.xacro"/>
-    </xacro:if>
-    <xacro:unless value = "$(arg use_ros2_control)">
-        <xacro:include filename="gazebo_control.xacro"/>
-    </xacro:unless>
+    <!-- <xacro:include filename="gazebo_control.xacro"/> -->
+    <xacro:include filename="ros2_control.xacro"/>
     <xacro:include filename="lidar.xacro"/>
 </robot>

File: install/dojo/share/dojo/description/robot_core.xacro (robot description, xacro)
@@ -47,5 +47,5 @@
         <child link="chassis"/>
         <origin xyz="${-wheel_offset_x} 0 ${-wheel_offset_z}"/>
-        <origin xyz="${-wheel_offset_x} 0 ${-wheel_offset_z}" rpy="0 0 ${pi}"/>
+        <!-- <origin xyz="${-wheel_offset_x} 0 ${-wheel_offset_z}" rpy="0 0 ${pi}"/> -->
     </joint>
     <link name="chassis">

File: install/dojo/share/dojo/description/ros2_control.xacro (robot description, xacro)
@@ -1,38 +1,15 @@
 <?xml version="1.0"?>
 <robot xmlns:xacro="http://www.ros.org/wiki/xacro">
-    <xacro:unless value="$(arg sim_mode)">
-        <ros2_control name="RealRobot" type="system">
+    <ros2_control name="RealRobot" type="system">
             <hardware>
-                <plugin>diffdrive_arduino/DiffDriveArduinoHardware</plugin>
+                <plugin>diffdrive_arduino/DiffDriveArduino</plugin>
                 <param name="left_wheel_name">left_wheel_joint</param>
                 <param name="right_wheel_name">right_wheel_joint</param>
                 <param name="loop_rate">30</param>
-                <param name="device">/dev/ACM0</param>
+                <param name="device">/dev/arduino</param>
                 <param name="baud_rate">57600</param>
-                <param name="timeout_ms">1000</param>
-                <param name="enc_counts_per_rev">1980</param>
-            </hardware>
-            <joint name="left_wheel_joint">
-                <command_interface name="velocity">
-                    <param name="min">-10</param>
-                    <param name="max">10</param>
-                </command_interface>
-                <state_interface name="position"/>
-                <state_interface name="velocity"/>
-            </joint>
-            <joint name="right_wheel_joint">
-                <command_interface name="velocity">
-                    <param name="min">-10</param>
-                    <param name="max">10</param>
-                </command_interface>
-                <state_interface name="position"/>
-                <state_interface name="velocity"/>
-            </joint>
-        </ros2_control>
-    </xacro:unless>
-    <xacro:if value="$(arg sim_mode)">
-        <ros2_control name="GazeboSystem" type="system">
-            <hardware>
-                <plugin>gazebo_ros2_control/GazeboSystem</plugin>
+                <param name="timeout">1000</param>
+                <!-- <param name="enc_counts_per_rev">1980</param> -->
+                <param name="enc_counts_per_rev">1135</param>
             </hardware>
             <joint name="left_wheel_joint">
@@ -53,9 +30,28 @@
             </joint>
         </ros2_control>
-    </xacro:if>
+    <!-- <ros2_control name="GazeboSystem" type="system">
+        <hardware>
+            <plugin>gazebo_ros2_control/GazeboSystem</plugin>
+        </hardware>
+        <joint name="left_wheel_joint">
+            <command_interface name="velocity">
+                <param name="min">-10</param>
+                <param name="max">10</param>
+            </command_interface>
+            <state_interface name="velocity"/>
+            <state_interface name="position"/>
+        </joint>
+        <joint name="right_wheel_joint">
+            <command_interface name="velocity">
+                <param name="min">-10</param>
+                <param name="max">10</param>
+            </command_interface>
+            <state_interface name="velocity"/>
+            <state_interface name="position"/>
+        </joint>
+    </ros2_control> -->
     <gazebo>
         <plugin name="gazebo_ros2_control" filename="libgazebo_ros2_control.so">
-            <parameters>$(find articubot_one)/config/my_controllers.yaml</parameters>
-            <parameters>$(find articubot_one)/config/gaz_ros2_ctl_use_sim.yaml</parameters>
+            <parameters>$(find dojo)/config/my_controllers.yaml</parameters>
         </plugin>
     </gazebo>
